Commit message: Added new 3D models to gazebo and moveit, and 'run' script

File: denso_robot_descriptions/vs_6577_b_description/vs_6577_b.urdf (robot description, URDF)
Before this commit: robot vs_6577_b, 8 links, 7 joints
Links:
- added link camera, mass 1; collision mesh filename=package://denso_robot_descriptions/vs_6577_b_description/ca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 scale=1 1 1; visual mesh filename=package://denso_robot_descriptions/vs_6577_b_description/ca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 scale=1 1 1
Joints:
- added joint camera_joint: type fixed, parent J6, child camera, origin xyz=0.000000 0.000000 0.000000 rpy=0.000000 0.000000 3.93000

Commit message: orientation working properly, tentative joint constraint, changed origin in camera 3d model

File: denso_robot_descriptions/vs_6577_b_description/vs_6577_b.urdf (robot description, URDF)
Before this commit: robot vs_6577_b, 9 links, 8 joints
Joints:
- joint camera_joint: origin xyz=0.000000 0.000000 0.000000 rpy=0.000000 0.000000 3.93000 -> xyz=-0.033000 -0.033000 0.115000 rpy=0.000000 -1.570796 0.785398

Commit message: camera projection, yet another new camera model

File: denso_robot_descriptions/vs_6577_b_description/vs_6577_b.urdf (robot description, URDF)
Before this commit: robot vs_6577_b, 9 links, 8 joints
Joints:
- joint camera_joint: origin xyz=-0.033000 -0.033000 0.115000 rpy=0.000000 -1.570796 0.785398 -> xyz=0.033 0.033 0.115 rpy=0.000000 0 -0.785398

Commit message: camera projection working in sim, possibly the last new camera model

File: denso_robot_descriptions/vs_6577_b_description/vs_6577_b.urdf (robot description, URDF)
Before this commit: robot vs_6577_b, 9 links, 8 joints
Joints:
- joint camera_joint: origin xyz=0.033 0.033 0.115 rpy=0.000000 0 -0.785398 -> xyz=0.033000 0.033000 0.115000 rpy=0.000000 0  2.356194

Commit message: everything is broken

File: denso_robot_descriptions/vs_6577_b_description/vs_6577_b.urdf (robot description, URDF)
Before this commit: robot vs_6577_b, 9 links, 8 joints
Joints:
- joint camera_joint: origin xyz=0.033000 0.033000 0.115000 rpy=0.000000 0  2.356194 -> xyz=0.033000 0.033000 0.070000 rpy=0.000000 0  2.356194

Commit message: new camera bracket

File: denso_robot_descriptions/vs_6577_b_description/vs_6577_b.urdf (robot description, URDF)
Before this commit: robot vs_6577_b, 9 links, 8 joints
Joints:
- joint camera_joint: origin xyz=0.033000 0.033000 0.070000 rpy=0.000000 0  2.356194 -> xyz=0.033000 0.033000 0.0765 rpy=0.000000 0  2.356194

Commit message: slightly offsetting the camera model improved performance

File: denso_robot_descriptions/vs_6577_b_description/vs_6577_b.urdf (robot description, URDF)
Before this commit: robot vs_6577_b, 9 links, 8 joints
Joints:
- joint camera_joint: origin xyz=0.033000 0.033000 0.0765 rpy=0.000000 0  2.356194 -> xyz=0.028000 0.033000 0.0765 rpy=0.000000 0  2.356194

Commit message: added a couple of files to aid in manual calibration

File: denso_robot_descriptions/vs_6577_b_description/vs_6577_b.urdf (robot description, URDF)
Before this commit: robot vs_6577_b, 9 links, 8 joints
Joints:
- joint camera_joint: origin xyz=0.028000 0.033000 0.0765 rpy=0.000000 0  2.356194 -> xyz=0.032775 0.033025 0.0765 rpy=0.000000 0  2.356194

Commit message: added handeye calibration scripts, refactoring

File: denso_robot_descriptions/vs_6577_b_description/vs_6577_b.urdf (robot description, URDF)
Before this commit: robot vs_6577_b, 9 links, 8 joints
Joints:
- joint camera_joint: origin xyz=0.032775 0.033025 0.0765 rpy=0.000000 0  2.356194 -> xyz=0.032775 0.033025 0.0765 rpy=0 0  2.356194
